File: discovery/pcb/discovery.kicad_sch (KiCad schematic)
At the start: 31 parts, among them J1 USB_C_Receptacle_USB2.0_16P, J2 BM03B-SRSS-TBLFSN, SW1 SW_Push, SW2 SW_Push, SW3 SW_SPST, U1 RP2350_60QFN, U2 USBLC6-2SC6, U3 AP2114H-3.3TRG1, U4 W25Q32JVZP, X1 ABM8-272-T3

Commit message: add rp2350 project
Parts:
- removed SW3: SW_SPST, symbol Switch:SW_SPST
- added 5V_PWR1: RED LED, LED_SMD:LED_0603_1608Metric, symbol Device:LED
- added C10, C11, C13, C14, C15, C16, C5, C7: 100n, Capacitor_SMD:C_0402_1005Metric, symbol Device:C
- added C6: 4.7u, Capacitor_SMD:C_0402_1005Metric, symbol Device:C
- added R12: 1k, Resistor_SMD:R_0402_1005Metric, symbol Device:R
- added R3: 220, Resistor_SMD:R_0402_1005Metric, symbol Device:R
- BOOT1: renamed from SW1; footprint (none) -> Button_Switch_SMD:SW_Push_1P1T_XKB_TS-1187A; LCSC (none) -> C318884
- C1: renamed from C7; footprint Capacitor_SMD:C_0402_1005Metric -> footprints:C_0402_1005Metric_small_pads; LCSC (none) -> C23733
- C12: renamed from C1; LCSC (none) -> C23733
- C2: renamed from C6; footprint Capacitor_SMD:C_0402_1005Metric -> footprints:C_0402_1005Metric_small_pads; LCSC (none) -> C23733
- C3: renamed from C8; LCSC (none) -> C23733
- C8: renamed from C2; LCSC (none) -> C23733
- C9: value C -> 100n; footprint (none) -> Capacitor_SMD:C_0402_1005Metric; LCSC (none) -> C1525
- FB1: footprint Inductor_SMD:L_0402_1005Metric -> LED_SMD:LED_0603_1608Metric; LCSC (none) -> C14709
- R1: renamed from R9; LCSC (none) -> C25105
- R4: renamed from R1; LCSC (none) -> C25905
- R5: renamed from R2; LCSC (none) -> C25905
- R6: renamed from R3; LCSC (none) -> C25100
- R7: renamed from R4; LCSC (none) -> C25100
- RUN1: renamed from SW2; footprint (none) -> Button_Switch_SMD:SW_Push_1P1T_XKB_TS-1187A; LCSC (none) -> C318884
- U2: LCSC (none) -> C7519
- renumbered C4 to C17, C5 to C18, C3 to C4, R8 to R10, R7 to R11, R5 to R2, R6 to R8, R10 to R9, U4 to U1, U1 to U4
Connections:
- net SW_VBUS_IN is gone; now on net VBUS: FB1.2
- net +1V1: now also U4.23 (DVDD), U4.39 (DVDD), U4.6 (DVDD), C5.1, C6.1, C7.1
- net +3V3: now also C9.1, U4.1 (IOVDD), U4.11 (IOVDD), U4.20 (IOVDD), U4.30 (IOVDD), U4.38 (IOVDD), U4.44 (ADC_AVDD), U4.45 (IOVDD), U4.53 (USB_OTP_VDD), U4.54 (QSPI_IOVDD), C10.1, C11.1, C13.1, C14.1, C15.1, C16.1
- net GND: now also C9.2, 5V_PWR1.1 (K), C10.2, C11.2, C13.2, C14.2, C15.2, C16.2, C5.2, C6.2, C7.2
- net VBUS: now also R3.2
- net XOUT: now also R12.2; no longer C18.1, X1.3
- new net: 5V_PWR1.2 (A), R3.1
- new net: C18.1, R12.1, X1.3
Other:
- note added: "Buttons"
- note removed: "Power Switch"
- moved on the sheet: C9, FB1, J1, U2
